File: ISO_3v3.kicad_sch (KiCad schematic)
At the start: 10 parts, among them U2 LD1117S33TR_SOT223, U3 NXE2S0505MC

Commit message: Update Power design - 29 October 2026, DRC clean
Parts:
- removed D1: Yellow-green, LED_SMD:LED_1206_3216Metric, symbol LED:LD271
- removed R1: 470Ω, Resistor_SMD:R_1206_3216Metric_Pad1.30x1.75mm_HandSolder, symbol Common_Components:R_US
- added R8: 100Ω, Resistor_SMD:R_1206_3216Metric_Pad1.30x1.75mm_HandSolder, symbol Common_Components:R_US
- C2: value 10µF -> 22µF; footprint Capacitor_SMD:C_1210_3225Metric_Pad1.33x2.70mm_HandSolder -> Capacitor_Tantalum_SMD:CP_EIA-3216-18_Kemet-A; ESR (none) -> 3 ohm maximum at 100kHz; LCSC C307584 -> C503893; Manufacturer KEMET -> TORCH; Manufacturer's Part Number C1210C106K5RACTU -> CA45-A-10V-22uF-K; Package (none) -> CASE-A-3216-16(mm); Polarity (none) -> +; Review Notes (none) -> LD1117 fixed-output application uses 100nF input and at lea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; Tolerance (none) -> 10%; Vendor 1 Digikey -> JLCPCB; Vendor 1 Cost (ea) 0.24 -> (none); Vendor 1 Order Code 399-C1210C106K5RACTUCT-ND -> C503893; Voltage Rating 16V -> 10V
- C4: LCSC C237223 -> C29823; Manufacturer Walsin Technology Corporation -> FH; Manufacturer's Part Number 1206B475K160CT -> 1206B475K500NT; Material Ceramic (X7R) -> X7R; Package (none) -> 1206; Review Notes (none) -> 4.7uF 50V X7R +/-10%; JLC Basic input filter capacitor for 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; Vendor 1 Digikey -> JLCPCB; Vendor 1 Cost (ea) - -> (none); Vendor 1 Order Code 1292-1206B475K160CTTR-ND -> C29823; Voltage Rating 16V -> 50V
- C5: Manufacturer KEMET -> Samsung Electro-Mechanics; Manufacturer's Part Number C1206C104K5RACTU -> CL31B104KBCNNNC; Package (none) -> 1206; Review Notes (none) -> 100nF 50V X7R 10%; JLC Basic candidate.; Vendor 1 Digikey -> JLCPCB; Vendor 1 Cost (ea) 0.08 -> (none); Vendor 1 Order Code 399-C1206C104K5RACTUCT-ND -> C24497
- C6: footprint Capacitor_SMD:C_1210_3225Metric_Pad1.33x2.70mm_HandSolder -> Capacitor_SMD:C_1206_3216Metric_Pad1.33x1.80mm_HandSolder; LCSC C307584 -> C13585; Manufacturer KEMET -> Samsung Electro-Mechanics; Manufacturer's Part Number C1210C106K5RACTU -> CL31A106KBHNNNE; Material Tantalum -> X5R; Package (none) -> 1206; Review Notes (none) -> 10uF 50V X5R 10%; JLC Basic candidate. Check effective capa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; Vendor 1 Digikey -> JLCPCB; Vendor 1 Cost (ea) 0.24 -> (none); Vendor 1 Order Code 399-C1210C106K5RACTUCT-ND -> C13585; Voltage Rating 16V -> 50V
- L3: Current Rating (none) -> 1A; DC Resistance (none) -> 0.325 ohm; Package (none) -> SMD,4x4mm; Review Notes (none) -> Retained existing 4x4mm input inductor. Allow approximately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; Saturation Current (none) -> 1.1A
- L4: footprint Common_Components:IND_8400_84XXXC_MUR -> Common_Components:L_Sunlord_SWPA5040; Current Rating (none) -> 1.5A; DC Resistance (none) -> 0.168 ohm max; LCSC C341013 -> C68434; Manufacturer YJYCOIN -> Sunlord; Manufacturer's Part Number YNR4030-220M -> SWPA5040S220MT; Package (none) -> SMD,5x5mm; Review Notes (none) -> 22uH output filter: 67.2mV maximum resistive drop at 400mA.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; Saturation Current (none) -> 1.6A minimum threshold; Vendor 1 (none) -> JLCPCB; Vendor 1 Order Code (none) -> C68434
- U2: value LD1117S33TR_SOT223 -> LD1117S33TR; Manufacturer (none) -> STMicroelectronics; Manufacturer's Part Number (none) -> LD1117S33TR; Package (none) -> SOT-223; Review Notes (none) -> Retained ST LD1117S33TR fixed 3.3V regulator. SOT223 pins 1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; Vendor 1 (none) -> JLCPCB; Vendor 1 Order Code (none) -> C86781
- U3: Manufacturer (none) -> Murata Electronics; Manufacturer's Part Number (none) -> NXE2S0505MC-R7; Package (none) -> SMD-5P,12.7x10.4mm; Review Notes (none) -> JLC catalogue part verified. Rated OUTPUT current 400mA; su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; Vendor 1 (none) -> JLCPCB; Vendor 1 Order Code (none) -> C5817088
Connections:
- net ISO_3v3_LDO: now also U2.2 (VO); no longer U2.3 (VI)
- net ISO_RET: now also U3.7 (-VOUT), R8.1; no longer U3.1 (-VIN)
- net at C4.1, L3.1: now also U3.3 (+VIN); no longer U3.8 (+VOUT)
- net at C5.2, C6.1, L4.1: now also U2.3 (VI), R8.2; no longer U2.2 (VO)
- net at L4.2: now also U3.8 (+VOUT); no longer U3.3 (+VIN)
- net EXT_RET_AUX renamed EXT_RET
- net EXT_RET: now also U3.1 (-VIN); no longer U3.7 (-VOUT)
Other:
- note added: "Load resistor guarentees DC:DC convertor minimum load requirement is met ≈ 50mA"
- moved on the sheet: C2, C5
