File: ISO_5v0.kicad_sch (KiCad schematic)
At the start: 7 parts, among them U1 NXE2S0505MC

Commit message: Update Power design - 29 October 2026, DRC clean
Parts:
- removed D2: Yellow-green, LED_SMD:LED_1206_3216Metric, symbol LED:LD271
- removed R2: 470Ω, Resistor_SMD:R_1206_3216Metric_Pad1.30x1.75mm_HandSolder, symbol Common_Components:R_US
- added R7: 100Ω, Resistor_SMD:R_1206_3216Metric_Pad1.30x1.75mm_HandSolder, symbol Common_Components:R_US
- C1: LCSC C237223 -> C29823; Manufacturer Walsin Technology Corporation -> FH; Manufacturer's Part Number 1206B475K160CT -> 1206B475K500NT; Material Ceramic (X7R) -> X7R; Package (none) -> 1206; Review Notes (none) -> 4.7uF 50V X7R +/-10%; JLC Basic input filter capacitor for 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; Vendor 1 Digikey -> JLCPCB; Vendor 1 Cost (ea) - -> (none); Vendor 1 Order Code 1292-1206B475K160CTTR-ND -> C29823; Voltage Rating 16V -> 50V
- C3: footprint Capacitor_SMD:C_1210_3225Metric_Pad1.33x2.70mm_HandSolder -> Capacitor_SMD:C_1206_3216Metric_Pad1.33x1.80mm_HandSolder; LCSC C307584 -> C13585; Manufacturer KEMET -> Samsung Electro-Mechanics; Manufacturer's Part Number C1210C106K5RACTU -> CL31A106KBHNNNE; Material Tantalum -> X5R; Package (none) -> 1206; Review Notes (none) -> 10uF 50V X5R 10%; JLC Basic candidate. Check effective capa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; Vendor 1 Digikey -> JLCPCB; Vendor 1 Cost (ea) 0.24 -> (none); Vendor 1 Order Code 399-C1210C106K5RACTUCT-ND -> C13585; Voltage Rating 16V -> 50V
- L1: Current Rating (none) -> 1A; DC Resistance (none) -> 0.325 ohm; Package (none) -> SMD,4x4mm; Review Notes (none) -> Retained existing 4x4mm input inductor. Allow approximately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; Saturation Current (none) -> 1.1A
- L2: footprint Common_Components:IND_8400_84XXXC_MUR -> Common_Components:L_Sunlord_SWPA5040; Current Rating (none) -> 1.5A; DC Resistance (none) -> 0.168 ohm max; LCSC C341013 -> C68434; Manufacturer YJYCOIN -> Sunlord; Manufacturer's Part Number YNR4030-220M -> SWPA5040S220MT; Package (none) -> SMD,5x5mm; Review Notes (none) -> 22uH output filter: 67.2mV maximum resistive drop at 400mA.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; Saturation Current (none) -> 1.6A minimum threshold; Vendor 1 (none) -> JLCPCB; Vendor 1 Order Code (none) -> C68434
- U1: Manufacturer (none) -> Murata Electronics; Manufacturer's Part Number (none) -> NXE2S0505MC-R7; Package (none) -> SMD-5P,12.7x10.4mm; Review Notes (none) -> JLC catalogue part verified. Rated OUTPUT current 400mA; su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; Vendor 1 (none) -> JLCPCB; Vendor 1 Order Code (none) -> C5817088
Connections:
- net EXT_RET: now also U1.1 (-VIN); no longer U1.7 (-VOUT)
- net ISO_5v0: now also R7.2
- net ISO_RET: now also U1.7 (-VOUT), R7.1; no longer U1.1 (-VIN)
- net at C1.1, L1.1: now also U1.3 (+VIN); no longer U1.8 (+VOUT)
- net at L2.2: now also U1.8 (+VOUT); no longer U1.3 (+VIN)
Other:
- note added: "50mA minimum"
- note added: "Load resistor guarentees DC:DC convertor minimum load requirement is met ≈ 50mA"
